File: pcb.kicad_pcb (KiCad board)
At the start: 4 copper layers, 26 x 25.6 mm, 64 parts, among them J2 Conn_ARM_JTAG_SWD_10, P1 USB_C_Plug, Q1 CJE3139K, Q2 CJE3139K, Q5 2N7002, Q6 2N7002, SW1 SW_Push, U1 WE-TVS-82400102, U2 STM32F103C8T6, U6 74LVC2T45DC, U7 74LVC2T45DC, U8 74LVC2T45DC, U9 AP2112K-3.3, Y1 8MHz

Commit message: Corrected USB resistors
Parts:
- removed R2: 5.1k, Resistor_SMD:R_0402_1005Metric
Connections:
- P1 pad B5: Net-(P1-VCONN) -> unconnected-(P1-VCONN-PadB5)
Routing:
- net Net-(P1-VCONN): track 3.71 -> 0.00 mm, vias 1 -> 0
- net GND: track 78.6 -> 77.6 mm
Other:
- board text added: "rev 1 Nov.2023"
- board text removed: "rev 0.1 June 2023"
