File: pcb.kicad_sch (KiCad schematic)
At the start: 63 parts, among them J2 Conn_ARM_JTAG_SWD_10, P1 USB_C_Plug, Q1 CJE3139K, Q2 CJE3139K, Q5 2N7002, Q6 2N7002, SW1 SW_Push, U1 WE-TVS-82400102, U3 STM32F103C8T6, U6 74LVC2T45DC, U7 74LVC2T45DC, U8 74LVC2T45DC, U9 AP2112K-3.3, Y1 8MHz

Commit message: Corrected USB resistors
Parts:
- removed R2: 5.1k, Resistor_SMD:R_0402_1005Metric, symbol Device:R_Small
Connections:
- no-connect marks 31 -> 32
Changed lines of the file:
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@@
   (junction (at 59.69 142.24) (diameter 0) (color 0 0 0 0)
   )
-  (junction (at 54.61 45.72) (diameter 0) (color 0 0 0 0)
-  )
   (junction (at 107.95 40.64) (diameter 0) (color 0 0 0 0)
   )
@@
   (no_connect (at 83.82 223.52))
   (no_connect (at 83.82 193.04))
+  (no_connect (at 45.72 48.26))
   (no_connect (at 45.72 91.44))
   (no_connect (at 83.82 213.36))
@@
     (stroke (width 0) (type default))
   )
-  (wire (pts (xy 54.61 48.26) (xy 53.34 48.26))
-    (stroke (width 0) (type default))
-  )
   (wire (pts (xy 135.89 49.53) (xy 135.89 48.26))
     (stroke (width 0) (type default))
@@
     (stroke (width 0) (type default))
   )
-  (wire (pts (xy 54.61 45.72) (xy 59.69 45.72))
-    (stroke (width 0) (type default))
-  )
   (wire (pts (xy 71.12 66.04) (xy 71.12 55.88))
     (stroke (width 0) (type default))
@@
     (stroke (width 0) (type default))
   )
-  (wire (pts (xy 53.34 45.72) (xy 54.61 45.72))
+  (wire (pts (xy 53.34 45.72) (xy 59.69 45.72))
     (stroke (width 0) (type default))
   )
@@
     (stroke (width 0) (type default))
   )
-  (wire (pts (xy 48.26 48.26) (xy 45.72 48.26))
-    (stroke (width 0) (type default))
-  )
   (wire (pts (xy 302.26 149.86) (xy 302.26 152.4))
     (stroke (width 0) (type default))
@@
     (stroke (width 0) (type default))
   )
-  (wire (pts (xy 54.61 45.72) (xy 54.61 48.26))
-    (stroke (width 0) (type default))
-  )
   (polyline (pts (xy 209.55 214.63) (xy 261.62 214.63))
     (stroke (width 0) (type default))
@@
         )
       )
-    )
-  )
-  (symbol (lib_id "Device:R_Small") (at 50.8 48.26 90) (mirror x) (unit 1)
-    (in_bom yes) (on_board yes) (dnp no)
-    (property "Reference" "R2" (at 48.26 50.8 90)
-      (effects (font (size 1.27 1.27)))
-    )
-    (property "Value" "5.1k" (at 53.34 50.8 90)
-      (effects (font (size 1.27 1.27)))
-    )
-    (property "Footprint" "Resistor_SMD:R_0402_1005Metric" (at 50.8 48.26 0)
-      (effects (font (size 1.27 1.27)) hide)
-    )
-    (property "Datasheet" "~" (at 50.8 48.26 0)
-      (effects (font (size 1.27 1.27)) hide)
-    )
-    (property "LCSC" "C881131" (at 50.8 48.26 0)
-      (effects (font (size 1.27 1.27)) hide)
-    )
-    (pin "1")
-    (pin "2")
-    (instances
-      (project "pcb"
-        (path "/74bf6178-dca6-4427-901b-44badacb7eee"
-          (reference "R2") (unit 1)
-        )
-      )
-      (project "framework_logic_analyzer"
-        (path "/cec59c69-8f0d-4d06-8fee-6cd1bb72d09c/2799dde1-a67f-418b-93ec-27396881451b"
-          (reference "R2") (unit 1)
-        )
-      )
